File: Hardware/Prototypes/Screen/H497TLB01/Breakout/Breakout.kicad_pcb (KiCad board)
At the start: 2 copper layers, 3 parts, among them P1 DISPLAY-RPi, P2 TOUCH SCREEN

Commit message: Some work
Parts:
- removed P2: TOUCH SCREEN, Pin_Header_2.54mm:2x5-BOX_HEADER-TH-VERTICAL
- OLED1: moved to F.Cu
- P1: value DISPLAY-RPi -> CONN_01X40; footprint SMD-Connectors:FPC_0.5mm_22p-MOLEX_52437 -> SMD-Connectors:OMRON-XF2M-40
- moved P1 3.01 mm to (137.2, 45.0)
- moved OLED1 3.00 mm to (137.0, 51.0), turned to 0 degrees
Connections:
- OLED1 pad 11: (no net) -> /OLED_TE
- OLED1 pad 12: (no net) -> /OLED_RESX
- P1 pad 1: +3V3 -> GND
- P1 pad 11: /DSI_D2_P -> +3V3
- P1 pad 12: /DSI_D2_N -> GND
- P1 pad 13: GND -> /DSI_D3_N
- P1 pad 14: /DSI_CK_P -> /DSI_D3_P
- P1 pad 15: /DSI_CK_N -> GND
- P1 pad 16: GND -> /DSI_D0_N
- P1 pad 17: /DSI_D1_P -> /DSI_D0_P
- P1 pad 18: /DSI_D1_N -> GND
- P1 pad 19: GND -> /DSI_CK_N
- P1 pad 2: /TOUCH_I2C_SDA -> GND
- P1 pad 20: /DSI_D0_P -> /DSI_CK_P
- P1 pad 21: /DSI_D0_N -> GND
- P1 pad 22: (no net) -> /DSI_D1_N
- P1 pad 3: /TOUCH_I2C_SCL -> /TOUCH_GPIO_A4
- P1 pad 4: GND -> /TOUCH_RESX
- P1 pad 5: (no net) -> /TOUCH_I2C_SCL
- P1 pad 6: (no net) -> /TOUCH_I2C_SDA
- P1 pad 7: GND -> /TOUCH_INT
- P1 pad 8: /DSI_D3_P -> +1V8
- P1 pad 9: /DSI_D3_N -> +3V3
Routing:
- net GND: track 0.00 -> 31.2 mm, vias 0 -> 22
- net +1V8: track 0.00 -> 21.2 mm, vias 0 -> 2
- net +BATT: track 0.00 -> 18.2 mm, vias 0 -> 17
- net +3V3: track 0.00 -> 8.60 mm, vias 0 -> 4
- net /DSI_D3_P: track 0.00 -> 8.33 mm, vias 0 -> 2
- net /OLED_TE: track 0.00 -> 7.46 mm, vias 0 -> 2
- net /DSI_D0_N: track 0.00 -> 7.06 mm, vias 0 -> 2
- net /TOUCH_RESX: track 0.00 -> 6.36 mm
- net /TOUCH_I2C_SDA: track 0.00 -> 6.19 mm
- net /TOUCH_GPIO_A4: track 0.00 -> 6.19 mm, vias 0 -> 2
- net /TOUCH_I2C_SCL: track 0.00 -> 5.48 mm, vias 0 -> 2
- net /DSI_D2_P: track 0.07 -> 5.36 mm, vias 0 -> 2
- net /TOUCH_INT: track 0.00 -> 5.11 mm, vias 0 -> 2
- net /DSI_D1_N: track 0.00 -> 5.03 mm, vias 0 -> 2
- net /DSI_CK_P: track 0.00 -> 5.03 mm, vias 0 -> 2
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- added copper zone on In2.Cu, net +3V3
- added copper zone on In2.Cu, net +BATT
- added copper zone on B.Cu, net GND
- added copper zone on F.Cu, net GND
- added copper zone on In1.Cu, net GND
Other:
- board outline added: 26 x 13 mm
- copper layers 2 -> 4
- board text added: "H497TLB01 Breakout RasmusB 2015"
- board text added: "v1.0"
