File: Hardware/Prototypes/Screen/H497TLB01/Breakout/Breakout.sch (KiCad schematic (older format))
At the start: 3 parts, among them P1 DISPLAY-RPi, P2 TOUCH SCREEN

Commit message: Some work
Parts:
- removed P1: DISPLAY-RPi, SMD-Connectors:FPC_0.5mm_22p-MOLEX_52437, symbol CONN_01X22
- removed P2: TOUCH SCREEN, Pin_Header_2.54mm:2x5-BOX_HEADER-TH-VERTICAL, symbol CONN_01X10
- added P1: CONN_01X40, symbol CONN_01X40
Connections:
- net +1V8: now also P1.28 (P28), P1.8 (P8)
- net +3V3: now also P1.11 (P11), P1.9 (P9)
- net +BATT: now also P1.35 (P35), P1.36 (P36), P1.37 (P37), P1.38 (P38), P1.39 (P39)
- net DSI_CK_N: now also P1.19 (P19)
- net DSI_CK_P: now also P1.20 (P20)
- net DSI_D0_N: now also P1.16 (P16)
- net DSI_D0_P: now also P1.17 (P17)
- net DSI_D1_N: now also P1.22 (P22)
- net DSI_D1_P: now also P1.23 (P23)
- net DSI_D2_N: now also P1.25 (P25)
- net DSI_D2_P: now also P1.26 (P26)
- net DSI_D3_N: now also P1.13 (P13)
- net DSI_D3_P: now also P1.14 (P14)
- net GND: now also P1.1 (P1), P1.10 (P10), P1.12 (P12), P1.15 (P15), P1.18 (P18), P1.2 (P2), P1.21 (P21), P1.24 (P24), P1.27 (P27), P1.32 (P32), P1.33 (P33), P1.34 (P34), P1.40 (P40)
- net OLED_RESX: now also P1.29 (P29)
- net OLED_TE: now also P1.30 (P30)
- net TOUCH_GPIO_A4: now also P1.3 (P3)
- net TOUCH_I2C_SCL: now also P1.5 (P5)
- net TOUCH_I2C_SDA: now also P1.6 (P6)
- net TOUCH_INT: now also P1.7 (P7)
- net TOUCH_RESX: now also P1.4 (P4)
- no-connect marks 2 -> 1
