File: Hardware/Prototypes/Keyboard/PCB/Keyboard.sch (KiCad schematic (older format))
At the start: 21 parts, among them CON1 USB-MICRO-B, U1 ATMEGA32U4-QFN44, X1 CRYSTAL-4pin

Commit message: Added the first version of the keyboard prototype module
Parts:
- removed C3: 10n, SMD-DiscreteB:0402-1005, symbol C
- removed CON1: USB-MICRO-B, SMD-Connectors:USB-MICRO, symbol USB-MICRO-B
- added USB1: TO HOST, symbol USB-EDGE-CONNECTOR
Connections:
- net labels removed: GNDD
- wire segments 122 -> 143
- no-connect marks 4 -> 3
Other:
- moved on the sheet: F1

Commit message: More work on the keyboard
Also an attempt to make an I2C based keyboard
Parts:
- C1, C11, C12, C2, C4, C5, C6, C7, C8: footprint SMD-DiscreteB:0402-1005 -> SMD-DiscreteB:C-0402-1005
- C10, C9: value 22p -> 10p; footprint SMD-DiscreteB:0402-1005 -> SMD-DiscreteB:C-0402-1005
- R1, R2, R3: footprint SMD-DiscreteB:0402-1005 -> SMD-DiscreteB:R-0402-1005
- USB1: footprint (none) -> Edge-Connectors:USB_EDGE
- X1: value CRYSTAL-4pin -> ABM10-16.000MHZ-D30-T3
Connections:
- wire segments 143 -> 115
Other:
- moved on the sheet: R1, R2

Commit message: Keyboard update
Version 1.1
Parts:
- removed USB1: TO HOST, Edge-Connectors:USB_EDGE, symbol USB-EDGE-CONNECTOR
- added C12: 4n7, SMD-DiscreteB:C-0402-1005, symbol C
- added D1: STATUS, SMD-DiscreteB:LED-0402-1005, symbol Led_Small
- added P1: USB_OTG, SMD-Connectors:USB-MICRO-MOLEX-47491-0001, symbol USB_OTG
- added R4: 1M, SMD-DiscreteB:R-0402-1005, symbol R
- added R5: 1k, SMD-DiscreteB:R-0402-1005, symbol R_Small
- added SW1: RESET, SMD-Switches:KSR251GLFS, symbol SW_PUSH
- C10: value 10p -> 15p
- C8: renamed from C9; value 10p -> 15p
- F1: footprint SMD-DiscreteB:0603-1608 -> SMD-DiscreteB:F-0603-1608; Farnell (none) -> 1717227
- ISP1: footprint SMD-Connectors:ISP-PADS_1mm27 -> SMD-Connectors:ISP-PADS_2mm54
- KB1: Farnell (none) -> 2520146
- U1: Farnell (none) -> 2425127
- X1: Farnell (none) -> 2467762
- renumbered C12 to C11, C4 to C3, C5 to C4, C6 to C5, C7 to C6, C8 to C7, C11 to C9
Connections:
- net labels added: GNDPWR, LED, TMP
- wire segments 115 -> 130
- no-connect marks 3 -> 1
Other:
- moved on the sheet: C1, C10, C11, C2, C3, C4, C5, C6, C7, C8, C9, R1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

Commit message: Reverted to 2-layer board
Because it fits and is cheaper
Connections:
- net GND: now also KB1.1 (NC), KB1.22 (NC)
- net LED: no longer KB1.1 (NC)
- net ROW_01: now also U1.40 (PF1/ADC1); no longer U1.1 (PE6/INT.6/AIN0)
- net ROW_07: now also U1.1 (PE6/INT.6/AIN0); no longer U1.40 (PF1/ADC1)
- net TMP: no longer KB1.22 (NC)
Changed lines of the file:
@@
 Wire Bus Line
 	9500 2650 9500 4550
-Text Label 7150 4550 2    60   ~ 0
+Text Label 7150 4850 2    60   ~ 0
 ROW_01
 Text Label 7150 5050 2    60   ~ 0
@@
 Text Label 7150 4950 2    60   ~ 0
 ROW_06
-Text Label 7150 4850 2    60   ~ 0
+Text Label 7100 4550 2    60   ~ 0
 ROW_07
 Text Label 7150 4750 2    60   ~ 0
@@
 Wire Wire Line
 	7050 2350 6750 2350
-Text Label 9600 4750 0    60   ~ 0
-LED
-Wire Wire Line
-	9600 4850 10050 4850
-Text Label 9600 4850 0    60   ~ 0
-TMP
-Wire Wire Line
-	9600 4750 10050 4750
 $Comp
 L SW_PUSH SW1
@@
 	1    0    0    -1
 $EndComp
+Wire Wire Line
+	10050 4850 9850 4850
+Wire Wire Line
+	9850 4750 9850 4950
+$Comp
+L GND #PWR?
+U 1 1 57FBF30B
+P 9850 4950
+F 0 "#PWR?" H 9850 4700 50  0001 C CNN
+F 1 "GND" H 9850 4800 50  0000 C CNN
+F 2 "" H 9850 4950 50  0000 C CNN
+F 3 "" H 9850 4950 50  0000 C CNN
+	1    9850 4950
+	1    0    0    -1
+$EndComp
+Wire Wire Line
+	10050 4750 9850 4750
+Connection ~ 9850 4850
 $EndSCHEMATC

Commit message: Further stuff done to prepare for prototypes
Parts:
- removed F1: 500mA, SMD-DiscreteB:F-0603-1608, symbol FUSE
- added F1: 500mA, SMD-DiscreteB:F-0603-1608, symbol F_Small
- SW1: footprint SMD-Switches:KSR251GLFS -> SMD-Switches:ALPS-SKRMAAE010
Connections:
- net +5V: now also F1.2
- net +5VD renamed VBUS
- net VBUS: now also F1.1
Changed lines of the file:
@@
 LIBS:valves
 LIBS:Keyboard-cache
-EELAYER 25 0
+EELAYER 26 0
 EELAYER END
 $Descr A4 11693 8268
@@
 	7300 5150 7200 5250
 $Comp
-L +5V #PWR01
+L +5V #PWR11
 U 1 1 54DFCCB0
 P 5150 1400
-F 0 "#PWR01" H 5150 1250 60  0001 C CNN
+F 0 "#PWR11" H 5150 1250 60  0001 C CNN
 F 1 "+5V" H 5150 1540 60  0000 C CNN
 F 2 "" H 5150 1400 60  0000 C CNN
@@
 $EndComp
 $Comp
-L GND #PWR02
+L GND #PWR12
 U 1 1 54DFCF30
 P 5400 6150
-F 0 "#PWR02" H 5400 5900 60  0001 C CNN
+F 0 "#PWR12" H 5400 5900 60  0001 C CNN
 F 1 "GND" H 5400 6000 60  0000 C CNN
 F 2 "" H 5400 6150 60  0000 C CNN
@@
 $EndComp
 $Comp
-L +5V #PWR03
+L +5V #PWR13
 U 1 1 54DFC139
 P 5550 1400
-F 0 "#PWR03" H 5550 1250 60  0001 C CNN
+F 0 "#PWR13" H 5550 1250 60  0001 C CNN
 F 1 "+5V" H 5550 1540 60  0000 C CNN
 F 2 "" H 5550 1400 60  0000 C CNN
@@
 $EndComp
 $Comp
-L +5V #PWR04
+L +5V #PWR14
 U 1 1 54DFC147
 P 5850 1400
-F 0 "#PWR04" H 5850 1250 60  0001 C CNN
+F 0 "#PWR14" H 5850 1250 60  0001 C CNN
 F 1 "+5V" H 5850 1540 60  0000 C CNN
 F 2 "" H 5850 1400 60  0000 C CNN
@@
 $EndComp
 $Comp
-L +5V #PWR05
+L +5V #PWR1
 U 1 1 54DFC155
 P 850 950
-F 0 "#PWR05" H 850 800 60  0001 C CNN
+F 0 "#PWR1" H 850 800 60  0001 C CNN
 F 1 "+5V" H 850 1090 60  0000 C CNN
 F 2 "" H 850 950 60  0000 C CNN
@@
 $EndComp
 $Comp
-L GND #PWR06
+L GND #PWR2
 U 1 1 54DFC193
 P 850 1850
-F 0 "#PWR06" H 850 1600 60  0001 C CNN
+F 0 "#PWR2" H 850 1600 60  0001 C CNN
 F 1 "GND" H 850 1700 60  0000 C CNN
 F 2 "" H 850 1850 60  0000 C CNN
@@
 VARef
 $Comp
-L GND #PWR07
+L GND #PWR5
 U 1 1 54DFD489
 P 1650 5700
-F 0 "#PWR07" H 1650 5450 60  0001 C CNN
+F 0 "#PWR5" H 1650 5450 60  0001 C CNN
 F 1 "GND" H 1650 5550 60  0000 C CNN
 F 2 "" H 1650 5700 60  0000 C CNN
@@
 $EndComp
 $Comp
-L GND #PWR08
+L GND #PWR9
 U 1 1 54DFE17B
 P 4400 3800
-F 0 "#PWR08" H 4400 3550 60  0001 C CNN
+F 0 "#PWR9" H 4400 3550 60  0001 C CNN
 F 1 "GND" H 4400 3650 60  0000 C CNN
 F 2 "" H 4400 3800 60  0000 C CNN
@@
 $EndComp
 $Comp
-L GND #PWR09
+L GND #PWR8
 U 1 1 54DFE3E2
 P 3300 3800
-F 0 "#PWR09" H 3300 3550 60  0001 C CNN
+F 0 "#PWR8" H 3300 3550 60  0001 C CNN
 F 1 "GND" H 3300 3650 60  0000 C CNN
 F 2 "" H 3300 3800 60  0000 C CNN
@@
 $EndComp
 $Comp
-L +5V #PWR010
+L +5V #PWR6
 U 1 1 54DFF76F
 P 2550 4200
-F 0 "#PWR010" H 2550 4050 60  0001 C CNN
+F 0 "#PWR6" H 2550 4050 60  0001 C CNN
 F 1 "+5V" H 2550 4340 60  0000 C CNN
 F 2 "" H 2550 4200 60  0000 C CNN
 F 3 "" H 2550 4200 60  0000 C CNN
 	1    2550 4200
-	1    0    0    -1
-$EndComp
-$Comp
-L FUSE F1
-U 1 1 54DFFDA6
-P 2100 4350
-F 0 "F1" H 2200 4400 50  0000 C CNN
-F 1 "500mA" H 2100 4300 50  0000 R CNN
-F 2 "SMD-DiscreteB:F-0603-1608" H 2100 4350 60  0001 C CNN
-F 3 "" H 2100 4350 60  0000 C CNN
-F 4 "1717227" H 2100 4350 60  0001 C CNN "Farnell"
-	1    2100 4350
 	1    0    0    -1
 $EndComp
@@
 $EndComp
 $Comp
-L +5V #PWR011
+L +5V #PWR10
 U 1 1 54E0055F
 P 4450 2250
-F 0 "#PWR011" H 4450 2100 60  0001 C CNN
+F 0 "#PWR10" H 4450 2100 60  0001 C CNN
 F 1 "+5V" H 4450 2390 60  0000 C CNN
 F 2 "" H 4450 2250 60  0000 C CNN
@@
 RESET
 $Comp
-L +5V #PWR012
+L +5V #PWR15
 U 1 1 54E02417
 P 9200 1000
-F 0 "#PWR012" H 9200 850 60  0001 C CNN
+F 0 "#PWR15" H 9200 850 60  0001 C CNN
 F 1 "+5V" H 9200 1140 60  0000 C CNN
 F 2 "" H 9200 1000 60  0000 C CNN
@@
 MOSI
 $Comp
-L GND #PWR013
+L GND #PWR16
 U 1 1 54E025DE
 P 9200 1650
-F 0 "#PWR013" H 9200 1400 60  0001 C CNN
+F 0 "#PWR16" H 9200 1400 60  0001 C CNN
 F 1 "GND" H 9200 1500 60  0000 C CNN
 F 2 "" H 9200 1650 60  0000 C CNN
@@
 Text Label 7050 2550 2    60   ~ 0
 MOSI
-$Comp
-L +5VD #PWR014
-U 1 1 54E0ECE1
-P 1650 4200
-F 0 "#PWR014" H 1650 4050 60  0001 C CNN
-F 1 "+5VD" H 1650 4340 60  0000 C CNN
-F 2 "" H 1650 4200 60  0000 C CNN
-F 3 "" H 1650 4200 60  0000 C CNN
-	1    1650 4200
-	1    0    0    -1
-$EndComp
 Wire Wire Line
 	9600 2750 10050 2750
@@
 	4550 4550 3500 4550
 Wire Wire Line
-	2550 4200 2550 4350
-Wire Wire Line
-	1450 4350 1850 4350
+	2550 4350 2550 4200
+Wire Wire Line
+	1450 4350 2000 4350
 Wire Wire Line
 	3950 2750 4550 2750
 Wire Wire Line
-	2550 4350 2350 4350
+	2200 4350 2550 4350
 Connection ~ 4450 2750
 Wire Wire Line
@@
 Connection ~ 1650 5400
 $Comp
-L GNDPWR #PWR015
+L GNDPWR #PWR3
 U 1 1 5736425E
 P 1050 5700
-F 0 "#PWR015" H 1050 5500 50  0001 C CNN
+F 0 "#PWR3" H 1050 5500 50  0001 C CNN
 F 1 "GNDPWR" H 1050 5570 50  0000 C CNN
 F 2 "" H 1050 5650 50  0000 C CNN
@@
 	10650 5450 10650 5550
 $Comp
-L GND #PWR016
+L GND #PWR18
 U 1 1 57F3D630
 P 10650 5550
-F 0 "#PWR016" H 10650 5300 50  0001 C CNN
+F 0 "#PWR18" H 10650 5300 50  0001 C CNN
 F 1 "GND" H 10650 5400 50  0000 C CNN
 F 2 "" H 10650 5550 50  0000 C CNN
@@
 F 0 "SW1" H 3800 2860 50  0000 C CNN
 F 1 "RESET" H 3650 2670 50  0000 C CNN
-F 2 "SMD-Switches:KSR251GLFS" H 3650 2750 50  0001 C CNN
+F 2 "SMD-Switches:ALPS-SKRMAAE010" H 3650 2750 50  0001 C CNN
 F 3 "" H 3650 2750 50  0000 C CNN
 F 4 "2376538" H 3650 2750 60  0001 C CNN "Farnell"
@@
 	3250 2750 3250 2850
 $Comp
-L GND #PWR017
+L GND #PWR7
 U 1 1 57F3F6A7
 P 3250 2850
-F 0 "#PWR017" H 3250 2600 60  0001 C CNN
+F 0 "#PWR7" H 3250 2600 60  0001 C CNN
 F 1 "GND" H 3250 2700 60  0000 C CNN
 F 2 "" H 3250 2850 60  0000 C CNN
@@
 	9850 4750 9850 4950
 $Comp
-L GND #PWR?
+L GND #PWR17
 U 1 1 57FBF30B
 P 9850 4950
-F 0 "#PWR?" H 9850 4700 50  0001 C CNN
+F 0 "#PWR17" H 9850 4700 50  0001 C CNN
 F 1 "GND" H 9850 4800 50  0000 C CNN
 F 2 "" H 9850 4950 50  0000 C CNN
@@
 	10050 4750 9850 4750
 Connection ~ 9850 4850
+$Comp
+L VBUS #PWR4
+U 1 1 583354E1
+P 1650 4200
+F 0 "#PWR4" H 1650 4050 50  0001 C CNN
+F 1 "VBUS" H 1665 4373 50  0000 C CNN
+F 2 "" H 1650 4200 60  0000 C CNN
+F 3 "" H 1650 4200 60  0000 C CNN
+	1    1650 4200
+	1    0    0    -1
+$EndComp
+$Comp
+L F_Small F1
+U 1 1 58335A2B
+P 2100 4350
+F 0 "F1" H 2100 4535 50  0000 C CNN
+F 1 "500mA" H 2100 4444 50  0000 C CNN
+F 2 "SMD-DiscreteB:F-0603-1608" H 2100 4350 50  0001 C CNN
+F 3 "" H 2100 4350 50  0000 C CNN
+F 4 "1717227" H 2100 4350 60  0001 C CNN "Farnell"
+	1    2100 4350
+	1    0    0    -1
+$EndComp
 $EndSCHEMATC

Commit message: Major data dump
Parts:
- P1: footprint SMD-Connectors:USB-MICRO-MOLEX-47491-0001 -> SMD-Connectors:USB-MICRO-10104110-0001LF; symbol USB_OTG -> USB_OTG-RESCUE-Keyboard; Farnell 1568025 -> 2293753; Mouser (none) -> 649-10104110-0001LF
- SW1: value RESET -> RST
Connections:
- net D-: now reaches R1.2, U1.3 (D-)
- net D+: now reaches R2.1, U1.4 (D+)
- net BUS-: now reaches P1.2 (D-), R1.1
- net BUS+: now reaches P1.3 (D+), R2.2
Changed lines of the file:
@@
 	7300 5150 7200 5250
 $Comp
-L +5V #PWR11
+L +5V #PWR01
 U 1 1 54DFCCB0
 P 5150 1400
-F 0 "#PWR11" H 5150 1250 60  0001 C CNN
+F 0 "#PWR01" H 5150 1250 60  0001 C CNN
 F 1 "+5V" H 5150 1540 60  0000 C CNN
 F 2 "" H 5150 1400 60  0000 C CNN
@@
 $EndComp
 $Comp
-L GND #PWR12
+L GND #PWR02
 U 1 1 54DFCF30
 P 5400 6150
-F 0 "#PWR12" H 5400 5900 60  0001 C CNN
+F 0 "#PWR02" H 5400 5900 60  0001 C CNN
 F 1 "GND" H 5400 6000 60  0000 C CNN
 F 2 "" H 5400 6150 60  0000 C CNN
@@
 $EndComp
 $Comp
-L +5V #PWR13
+L +5V #PWR03
 U 1 1 54DFC139
 P 5550 1400
-F 0 "#PWR13" H 5550 1250 60  0001 C CNN
+F 0 "#PWR03" H 5550 1250 60  0001 C CNN
 F 1 "+5V" H 5550 1540 60  0000 C CNN
 F 2 "" H 5550 1400 60  0000 C CNN
@@
 $EndComp
 $Comp
-L +5V #PWR14
+L +5V #PWR04
 U 1 1 54DFC147
 P 5850 1400
-F 0 "#PWR14" H 5850 1250 60  0001 C CNN
+F 0 "#PWR04" H 5850 1250 60  0001 C CNN
 F 1 "+5V" H 5850 1540 60  0000 C CNN
 F 2 "" H 5850 1400 60  0000 C CNN
@@
 $EndComp
 $Comp
-L +5V #PWR1
+L +5V #PWR05
 U 1 1 54DFC155
 P 850 950
-F 0 "#PWR1" H 850 800 60  0001 C CNN
+F 0 "#PWR05" H 850 800 60  0001 C CNN
 F 1 "+5V" H 850 1090 60  0000 C CNN
 F 2 "" H 850 950 60  0000 C CNN
@@
 $EndComp
 $Comp
-L GND #PWR2
+L GND #PWR06
 U 1 1 54DFC193
 P 850 1850
-F 0 "#PWR2" H 850 1600 60  0001 C CNN
+F 0 "#PWR06" H 850 1600 60  0001 C CNN
 F 1 "GND" H 850 1700 60  0000 C CNN
 F 2 "" H 850 1850 60  0000 C CNN
@@
 VARef
 $Comp
-L GND #PWR5
+L GND #PWR07
 U 1 1 54DFD489
 P 1650 5700
-F 0 "#PWR5" H 1650 5450 60  0001 C CNN
+F 0 "#PWR07" H 1650 5450 60  0001 C CNN
 F 1 "GND" H 1650 5550 60  0000 C CNN
 F 2 "" H 1650 5700 60  0000 C CNN
@@
 $EndComp
 $Comp
-L GND #PWR9
+L GND #PWR08
 U 1 1 54DFE17B
 P 4400 3800
-F 0 "#PWR9" H 4400 3550 60  0001 C CNN
+F 0 "#PWR08" H 4400 3550 60  0001 C CNN
 F 1 "GND" H 4400 3650 60  0000 C CNN
 F 2 "" H 4400 3800 60  0000 C CNN
@@
 $EndComp
 $Comp
-L GND #PWR8
+L GND #PWR09
 U 1 1 54DFE3E2
 P 3300 3800
-F 0 "#PWR8" H 3300 3550 60  0001 C CNN
+F 0 "#PWR09" H 3300 3550 60  0001 C CNN
 F 1 "GND" H 3300 3650 60  0000 C CNN
 F 2 "" H 3300 3800 60  0000 C CNN
@@
 $EndComp
 $Comp
-L +5V #PWR6
+L +5V #PWR010
 U 1 1 54DFF76F
 P 2550 4200
-F 0 "#PWR6" H 2550 4050 60  0001 C CNN
+F 0 "#PWR010" H 2550 4050 60  0001 C CNN
 F 1 "+5V" H 2550 4340 60  0000 C CNN
 F 2 "" H 2550 4200 60  0000 C CNN
@@
 $EndComp
 $Comp
-L +5V #PWR10
+L +5V #PWR011
 U 1 1 54E0055F
 P 4450 2250
-F 0 "#PWR10" H 4450 2100 60  0001 C CNN
+F 0 "#PWR011" H 4450 2100 60  0001 C CNN
 F 1 "+5V" H 4450 2390 60  0000 C CNN
 F 2 "" H 4450 2250 60  0000 C CNN
@@
 RESET
 $Comp
-L +5V #PWR15
+L +5V #PWR012
 U 1 1 54E02417
 P 9200 1000
-F 0 "#PWR15" H 9200 850 60  0001 C CNN
+F 0 "#PWR012" H 9200 850 60  0001 C CNN
 F 1 "+5V" H 9200 1140 60  0000 C CNN
 F 2 "" H 9200 1000 60  0000 C CNN
@@
 MOSI
 $Comp
-L GND #PWR16
+L GND #PWR013
 U 1 1 54E025DE
 P 9200 1650
-F 0 "#PWR16" H 9200 1400 60  0001 C CNN
+F 0 "#PWR013" H 9200 1400 60  0001 C CNN
 F 1 "GND" H 9200 1500 60  0000 C CNN
 F 2 "" H 9200 1650 60  0000 C CNN
@@
 	7200 3850 6750 3850
 $Comp
-L USB_OTG P1
+L USB_OTG-RESCUE-Keyboard P1
 U 1 1 5727A357
 P 1150 4550
 F 0 "P1" H 1475 4425 50  0000 C CNN
 F 1 "USB_OTG" H 1150 4750 50  0000 C CNN
-F 2 "SMD-Connectors:USB-MICRO-MOLEX-47491-0001" V 1100 4450 50  0001 C CNN
+F 2 "SMD-Connectors:USB-MICRO-10104110-0001LF" V 1100 4450 50  0001 C CNN
 F 3 "" V 1100 4450 50  0000 C CNN
-F 4 "1568025" H 1150 4550 60  0001 C CNN "Farnell"
+F 4 "2293753" H 1150 4550 60  0001 C CNN "Farnell"
+F 5 "649-10104110-0001LF" H 1150 4550 60  0001 C CNN "Mouser"
 	1    1150 4550
 	0    -1   1    0
@@
 Connection ~ 1650 5400
 $Comp
-L GNDPWR #PWR3
+L GNDPWR #PWR014
 U 1 1 5736425E
 P 1050 5700
-F 0 "#PWR3" H 1050 5500 50  0001 C CNN
+F 0 "#PWR014" H 1050 5500 50  0001 C CNN
 F 1 "GNDPWR" H 1050 5570 50  0000 C CNN
 F 2 "" H 1050 5650 50  0000 C CNN
@@
 	10650 5450 10650 5550
 $Comp
-L GND #PWR18
+L GND #PWR015
 U 1 1 57F3D630
 P 10650 5550
-F 0 "#PWR18" H 10650 5300 50  0001 C CNN
+F 0 "#PWR015" H 10650 5300 50  0001 C CNN
 F 1 "GND" H 10650 5400 50  0000 C CNN
 F 2 "" H 10650 5550 50  0000 C CNN
@@
 P 3650 2750
 F 0 "SW1" H 3800 2860 50  0000 C CNN
-F 1 "RESET" H 3650 2670 50  0000 C CNN
+F 1 "RST" H 3650 2670 50  0000 C CNN
 F 2 "SMD-Switches:ALPS-SKRMAAE010" H 3650 2750 50  0001 C CNN
 F 3 "" H 3650 2750 50  0000 C CNN
@@
 	3250 2750 3250 2850
 $Comp
-L GND #PWR7
+L GND #PWR016
 U 1 1 57F3F6A7
 P 3250 2850
-F 0 "#PWR7" H 3250 2600 60  0001 C CNN
+F 0 "#PWR016" H 3250 2600 60  0001 C CNN
 F 1 "GND" H 3250 2700 60  0000 C CNN
 F 2 "" H 3250 2850 60  0000 C CNN
@@
 	9850 4750 9850 4950
 $Comp
-L GND #PWR17
+L GND #PWR017
 U 1 1 57FBF30B
 P 9850 4950
-F 0 "#PWR17" H 9850 4700 50  0001 C CNN
+F 0 "#PWR017" H 9850 4700 50  0001 C CNN
 F 1 "GND" H 9850 4800 50  0000 C CNN
 F 2 "" H 9850 4950 50  0000 C CNN
@@
 Connection ~ 9850 4850
 $Comp
-L VBUS #PWR4
+L VBUS #PWR018
 U 1 1 583354E1
 P 1650 4200
-F 0 "#PWR4" H 1650 4050 50  0001 C CNN
+F 0 "#PWR018" H 1650 4050 50  0001 C CNN
 F 1 "VBUS" H 1665 4373 50  0000 C CNN
 F 2 "" H 1650 4200 60  0000 C CNN
@@
 	1    0    0    -1
 $EndComp
+Text Label 2800 4450 0    60   ~ 0
+BUS-
+Text Label 2800 4550 0    60   ~ 0
+BUS+
+Text Label 3650 4450 0    60   ~ 0
+D-
+Text Label 3650 4550 0    60   ~ 0
+D+
 $EndSCHEMATC
