File: Hardware/Prototypes/Mainboard/Mainboard.kicad_pcb (KiCad board)
At the start: 4 copper layers, 16 parts, among them J1 USB_B_Micro, J2 LiPo, J3 BAT_V, J4 BAT_T, J5 +5V, U1 OSD3358-512M-BCB

Commit message: More work
Still on the power section. Next - clamping circuit!
Parts:
- added J6: I2C0, Connector_PinHeader_2.54mm:PinHeader_1x03_P2.54mm_Vertical, F.Cu at (156.2, 59.7)
- added JP1: PMIC_NRESET, Connector_PinHeader_2.54mm:PinHeader_1x02_P2.54mm_Vertical, F.Cu at (111.8, 83.8)
- added R1: 1k5, Resistor_SMD:R_0603_1608Metric, F.Cu at (169.1, 105.1)
- added R2: 1k5, Resistor_SMD:R_0603_1608Metric, F.Cu at (169.1, 102.5)
- added SW1: POWER, Button_Switch_SMD:SW_SPST_B3SL-1002P, F.Cu at (125.7, 88.9)
- added TP10: NINT, TestPoint:TestPoint_Pad_D1.0mm, F.Cu at (160.1, 65.0)
- added TP7: PWREN, TestPoint:TestPoint_Pad_D1.0mm, F.Cu at (160.1, 58.9)
- added TP8: LPGD, TestPoint:TestPoint_Pad_D1.0mm, F.Cu at (160.1, 61.9)
- added TP9: NWKP, TestPoint:TestPoint_Pad_D1.0mm, F.Cu at (163.1, 58.9)
- TP11: renamed from TP7; footprint TestPoint:TestPoint_Keystone_5015_Micro-Minature -> TestPoint:TestPoint_Pad_D1.0mm
- TP12: renamed from TP8; footprint TestPoint:TestPoint_Keystone_5015_Micro-Minature -> TestPoint:TestPoint_Pad_D1.0mm
- TP13: renamed from TP9; footprint TestPoint:TestPoint_Keystone_5015_Micro-Minature -> TestPoint:TestPoint_Pad_D1.0mm
- TP2, TP3, TP4, TP5, TP6: footprint TestPoint:TestPoint_Keystone_5015_Micro-Minature -> TestPoint:TestPoint_Pad_D1.0mm
- renumbered R1 to R3
Connections:
- U1 pad A18: Net-(U1-PadA18) -> /Power/PMIC_PB_IN
- U1 pad A19: Net-(U1-PadA19) -> /Power/PMIC_NRESET
- U1 pad D10: Net-(U1-PadD10) -> Net-(TP7-Pad1)
- U1 pad D13: Net-(U1-PadD13) -> Net-(TP8-Pad1)
- U1 pad D14: Net-(U1-PadD14) -> Net-(TP8-Pad1)
- U1 pad D9: Net-(U1-PadD9) -> Net-(TP7-Pad1)
- U1 pad G17: Net-(U1-PadG17) -> Net-(TP9-Pad1)
- U1 pad H17: Net-(U1-PadH17) -> Net-(TP9-Pad1)
- U1 pad J17: Net-(U1-PadJ17) -> Net-(TP10-Pad1)
- U1 pad K17: Net-(U1-PadK17) -> Net-(TP10-Pad1)
- U1 pad U7: Net-(U1-PadU7) -> /Power/I2C0_SDA
- U1 pad U8: Net-(U1-PadU8) -> /Power/I2C0_SCL
- U1 pad V7: Net-(U1-PadV7) -> /Power/I2C0_SDA
- U1 pad V8: Net-(U1-PadV8) -> /Power/I2C0_SCL
Routing:
- added copper zone on F.Cu, net GND
